File: hardware/Cyberboard.kicad_sch (KiCad schematic)
At the start: 69 parts, among them J1 Conn_01x20, J2 Conn_01x20, SW1 SW_Push, SW2 SW_Push, U1 SZYY0402Y_C434450, U10 XL-1005UBC_C22355736, U2 TPD2EUSB30, U3 NX2012SA-32.768KHZ-STD-MUB-2, U4 STM32WB55RGVx, U5 BQ24072RGT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

Commit message: started PCB
Connections:
- net GPIO24: now also U4.51 (PA10); no longer U4.57 (PA15)
- net GPIO25: now also U4.57 (PA15); no longer U4.58 (PC10)
- net GPIO26: now also U4.58 (PC10); no longer U4.59 (PC11)
- net GPIO27: now also U4.59 (PC11); no longer U4.60 (PC12)
- net GPIO28: now also U4.60 (PC12); no longer U4.61 (PD0)
- net GPIO29: now also U4.61 (PD0)
- net LED: now also U4.62 (PD1)
- net at C7.1, L1.2: now also U4.41 (VFBSMPS)
- no-connect marks 5 -> 7

Commit message: start routing
Parts:
- removed D1: PESD15VL1BA, Diode_SMD:D_SOD-323, symbol PCM_Diode_TVS_AKL:PESD15VL1BA
- C14, C17: footprint Capacitor_SMD:C_0603_1608Metric -> Capacitor_SMD:C_0402_1005Metric
- C25, C26: footprint Capacitor_SMD:C_0402_1005Metric -> Capacitor_SMD:C_0603_1608Metric
Connections:
- net I2C_SCL is gone; now on net BMP_SCL: R11.1, U8.2 (SCK)
- net I2C_SDA is gone; now on net BMP_SDA: R12.1, U8.4 (SDI)
- net GPIO16: now also U4.40 (PE4); no longer U4.38 (PB0)
- net GPIO18: now also U4.38 (PB0); no longer U4.40 (PE4)
- net GPIO26: now also U4.61 (PD0); no longer U4.58 (PC10)
- net GPIO27: now also U4.60 (PC12); no longer U4.59 (PC11)
- net GPIO28: now also U4.58 (PC10); no longer U4.60 (PC12)
- net GPIO29: now also U4.59 (PC11); no longer U4.61 (PD0)
- net ICM_CS: now also U4.62 (PD1); no longer U4.2 (PC13)
- net ICM_INT1: now also U7.4 (INT1)
- net ICM_INT2: no longer U7.4 (INT1)
- net LED: now also U4.2 (PC13); no longer U4.62 (PD1)

Commit message: add stuff
Parts:
- J1, J2: LCSC (none) -> C42431804
- R4: LCSC (none) -> C25082
- TP1, TP2, TP3, TP4, TP5: now left out of the parts list
- U4: LCSC (none) -> C401505
- U5: LCSC (none) -> C140288
Connections:
- net GPIO16: now also U4.38 (PB0); no longer U4.40 (PE4)
- net GPIO18: now also U4.40 (PE4); no longer U4.38 (PB0)
- net GPIO26: now also U4.58 (PC10); no longer U4.61 (PD0)
- net GPIO27: now also U4.59 (PC11); no longer U4.60 (PC12)
- net GPIO28: now also U4.60 (PC12); no longer U4.58 (PC10)
- net GPIO29: now also U4.61 (PD0); no longer U4.59 (PC11)

Commit message: final final bluetooth trace udpate
Parts:
- added R16: 4.7K, Resistor_SMD:R_0402_1005Metric, symbol Device:R
Connections:
- net +3.3V: now also R16.2
- net ICM_CS: now also R16.1
Changed lines of the file:
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@@
 	)
 	(junction
+		(at 394.97 90.17)
+		(diameter 0)
+		(color 0 0 0 0)
+	)
+	(junction
 		(at 66.04 241.3)
 		(diameter 0)
@@
 	)
 	(junction
+		(at 381 100.33)
+		(diameter 0)
+		(color 0 0 0 0)
+	)
+	(junction
 		(at 325.12 38.1)
 		(diameter 0)
@@
 	(wire
 		(pts
-			(xy 378.46 100.33) (xy 368.3 100.33)
+			(xy 391.16 100.33) (xy 381 100.33)
 		)
 		(stroke
@@
 	(wire
 		(pts
+			(xy 381 99.06) (xy 381 100.33)
+		)
+		(stroke
+			(width 0)
+			(type default)
+		)
+	)
+	(wire
+		(pts
 			(xy 393.7 163.83) (xy 382.27 163.83)
 		)
@@
 	(wire
 		(pts
+			(xy 381 90.17) (xy 381 91.44)
+		)
+		(stroke
+			(width 0)
+			(type default)
+		)
+	)
+	(wire
+		(pts
 			(xy 255.27 245.11) (xy 266.7 245.11)
 		)
@@
 	(wire
 		(pts
+			(xy 381 90.17) (xy 394.97 90.17)
+		)
+		(stroke
+			(width 0)
+			(type default)
+		)
+	)
+	(wire
+		(pts
 			(xy 219.71 167.64) (xy 219.71 171.45)
 		)
@@
 	(wire
 		(pts
+			(xy 381 100.33) (xy 368.3 100.33)
+		)
+		(stroke
+			(width 0)
+			(type default)
+		)
+	)
+	(wire
+		(pts
 			(xy 53.34 187.96) (xy 52.07 187.96)
 		)
@@
 	(wire
 		(pts
-			(xy 394.97 95.25) (xy 394.97 110.49)
+			(xy 394.97 90.17) (xy 394.97 110.49)
+		)
+		(stroke
+			(width 0)
+			(type default)
+		)
+	)
+	(wire
+		(pts
+			(xy 394.97 88.9) (xy 394.97 90.17)
 		)
 		(stroke
@@
 	)
 	(label "ICM_CS"
-		(at 378.46 100.33 180)
+		(at 391.16 100.33 180)
 		(effects
 			(font
@@
 	(symbol
 		(lib_id "Device:R")
+		(at 381 95.25 180)
+		(unit 1)
+		(exclude_from_sim no)
+		(in_bom yes)
+		(on_board yes)
+		(dnp no)
+		(property "Reference" "R16"
+			(at 384.556 93.98 0)
+			(effects
+				(font
+					(size 1.27 1.27)
+				)
+			)
+		)
+		(property "Value" "4.7K"
+			(at 384.556 96.266 0)
+			(effects
+				(font
+					(size 1.27 1.27)
+				)
+			)
+		)
+		(property "Footprint" "Resistor_SMD:R_0402_1005Metric"
+			(at 382.778 95.25 90)
+			(effects
+				(font
+					(size 1.27 1.27)
+				)
+				(hide yes)
+			)
+		)
+		(property "Datasheet" "~"
+			(at 381 95.25 0)
+			(effects
+				(font
+					(size 1.27 1.27)
+				)
+				(hide yes)
+			)
+		)
+		(property "Description" "Resistor"
+			(at 381 95.25 0)
+			(effects
+				(font
+					(size 1.27 1.27)
+				)
+				(hide yes)
+			)
+		)
+		(pin "2"
+		)
+		(pin "1"
+		)
+		(instances
+			(project "Cyberboard"
+				(path "/3bb22019-5160-4958-be00-a0bb623b71d1"
+					(reference "R16")
+					(unit 1)
+				)
+			)
+		)
+	)
+	(symbol
+		(lib_id "Device:R")
 		(at 313.69 181.61 90)
 		(unit 1)
@@
 	(symbol
 		(lib_id "power:+3.3V")
-		(at 394.97 95.25 0)
+		(at 394.97 88.9 0)
 		(unit 1)
 		(exclude_from_sim no)
@@
 		(dnp no)
 		(property "Reference" "#PWR056"
-			(at 394.97 99.06 0)
+			(at 394.97 92.71 0)
 			(effects
 				(font
@@
 		)
 		(property "Value" "+3.3V"
-			(at 394.97 91.44 0)
+			(at 394.97 85.09 0)
 			(effects
 				(font
@@
 		)
 		(property "Footprint" ""
-			(at 394.97 95.25 0)
+			(at 394.97 88.9 0)
 			(effects
 				(font
@@
 		)
 		(property "Datasheet" ""
-			(at 394.97 95.25 0)
+			(at 394.97 88.9 0)
 			(effects
 				(font
@@
 		)
 		(property "Description" "Power symbol creates a global label with name \"+3.3V\""
-			(at 394.97 95.25 0)
+			(at 394.97 88.9 0)
 			(effects
 				(font
