File: hardware/panel/Cyberboard_Panel.kicad_pcb (KiCad board)
At the start: 4 copper layers, 51 x 44 mm, 136 parts, among them J1 Conn_01x20, J2 Conn_01x20, SW1 SW_Push, SW2 SW_Push, U1 SZYY0402Y_C434450, U10 XL-1005UBC_C22355736, U2 TPD2EUSB30, U3 NX2012SA-32.768KHZ-STD-MUB-2, U4 STM32WB55RGVx, U5 BQ24072RGT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

Commit message: final final bluetooth trace udpate
Parts:
- added R16: 4.7K, Resistor_SMD:R_0402_1005Metric, F.Cu at (152.0, 36.0)
- added R16: 4.7K, Resistor_SMD:R_0402_1005Metric, F.Cu at (152.0, 59.0)
Routing:
- net Board_1-GND: track 25.9 -> 33.2 mm, vias 73 -> 85
- net Board_0-GND: track 25.9 -> 33.2 mm, vias 73 -> 85
- net Board_1-/ICM_CS: track 14.6 -> 16.1 mm
- net Board_0-/ICM_CS: track 14.6 -> 16.1 mm
- net Board_1-+3.3V: track 50.2 -> 50.7 mm, vias 18 -> 19
- net Board_0-+3.3V: track 50.2 -> 50.7 mm, vias 18 -> 19
